File: PCBs/TADPOL PCB/TADPOL PCB v2/TADPOL PCB v2.kicad_sch (KiCad schematic)
At the start: 13 parts

Commit message: PCB v2
Parts:
- added H1, H2, H3, H4: MountingHole, MountingHole:MountingHole_3.2mm_M3, symbol Mechanical:MountingHole
- BypassSwitch1: footprint (none) -> Connector_JST:JST_XH_B2B-XH-A_1x02_P2.50mm_Vertical
- D2: footprint (none) -> Package_TO_SOT_THT:TO-220-2_Vertical
- LiveVideo1: renamed from LiveVideo; footprint (none) -> Connector_JST:JST_XH_B5B-XH-A_1x05_P2.50mm_Vertical
- LoRa_Radio1: renamed from LoRa_Radio; footprint (none) -> Connector_JST:JST_XH_B4B-XH-A_1x04_P2.50mm_Vertical
- NichromeConnect1: renamed from NichromeConnector1; footprint (none) -> Connector_JST:JST_XH_B3B-XH-A_1x03_P2.50mm_Vertical
- NichromeConnect2: renamed from NichromeConnector2; footprint (none) -> Connector_JST:JST_XH_B3B-XH-A_1x03_P2.50mm_Vertical
- Power1: renamed from Power; footprint (none) -> Connector_JST:JST_XH_B2B-XH-A_1x02_P2.50mm_Vertical
- PowerOUT1: renamed from PowerOUT; footprint (none) -> Connector_JST:JST_XH_B2B-XH-A_1x02_P2.50mm_Vertical
- SensorBoard1: renamed from SensorBoard; footprint (none) -> Connector_JST:JST_XH_B4B-XH-A_1x04_P2.50mm_Vertical
- Servo1: footprint (none) -> Connector_JST:JST_XH_B3B-XH-A_1x03_P2.50mm_Vertical
- VoltageRegulator5V1: renamed from VoltageRegulator5V; footprint (none) -> Package_TO_SOT_THT:TO-220-3_Vertical
- VoltageRegulator6V1: renamed from VoltageRegulator6V; footprint (none) -> Package_TO_SOT_THT:TO-220-3_Vertical

Commit message: fixed scr pcb
Parts:
- removed D2: D, Package_TO_SOT_THT:TO-220-2_Vertical, symbol Device:D
- removed VoltageRegulator6V1: L7806, Package_TO_SOT_THT:TO-220-3_Vertical, symbol Regulator_Linear:L7806
- added SCR_Latchup: L7805, Package_TO_SOT_THT:TO-220-3_Vertical, symbol Regulator_Linear:L7805
- renumbered NichromeConnect1 to Servo2, NichromeConnect2 to Servo3
Connections:
- net +6V is gone; now on net +5V: Servo1.2 (Pin_2)
- net GND: now also SCR_Latchup.2 (GND)
- net VIN: now also SCR_Latchup.3 (OUT)
- net at BypassSwitch1.1 (Pin_1), Power1.1 (Pin_1): now also SCR_Latchup.1 (IN)
- net PWM_SERVO2: now reaches Teensy4.1.4 (PWM)
- net PWM_SERVO2: now also Servo2.2 (Pin_2)
- net PWM_SERVO3: now reaches Teensy4.1.5 (PWM)
- net PWM_SERVO3: now also Servo3.2 (Pin_2)
- net PWM_NICHROME1: no longer names the net of Teensy4.1.44 (PWM)
- net PWM_NICHROME1: no longer Servo2.2 (Pin_2)
- net PWM_NICHROME2: no longer names the net of Teensy4.1.43 (PWM)
- net PWM_NICHROME2: no longer Servo3.2 (Pin_2)
Other:
- moved on the sheet: VoltageRegulator5V1

Commit message: Updated PCB
Parts:
- removed SCR_Latchup: L7805, Package_TO_SOT_THT:TO-220-3_Vertical, symbol Regulator_Linear:L7805
- added BZ1: Buzzer, Buzzer_Beeper:Buzzer_12x9.5RM7.6, symbol Device:Buzzer
- added D1: Q_SCR_KAG, Package_TO_SOT_THT:TO-220-3_Vertical, symbol Device:Q_SCR_KAG
- added SerialConnect1: Conn_01x04_Socket, Connector_JST:JST_XH_B4B-XH-A_1x04_P2.50mm_Vertical, symbol Connector:Conn_01x04_Socket
- renumbered VoltageRegulator5V1 to VoltRegulator5V1
Connections:
- net +5V: now also Servo2.2 (Pin_2), Servo3.2 (Pin_2)
- net GND: now also BZ1.2 (-), SerialConnect1.1 (Pin_1)
- net PWM_SERVO2: now also Servo2.1 (Pin_1); no longer Servo2.2 (Pin_2)
- net PWM_SERVO3: now also Servo3.1 (Pin_1); no longer Servo3.2 (Pin_2)
- net VIN: now also D1.1 (K); no longer Servo2.1 (Pin_1), Servo3.1 (Pin_1)
- net at BypassSwitch1.1 (Pin_1), Power1.1 (Pin_1): now also D1.2 (A)
- net RX_SERIAL: now reaches Teensy4.1.1 (RX1)
- net RX_SERIAL: now also SerialConnect1.2 (Pin_2)
- net TX_SERIAL: now reaches Teensy4.1.2 (TX1)
- net TX_SERIAL: now also SerialConnect1.3 (Pin_3)
- net BUZZER: now reaches Teensy4.1.24 (PWM)
- net BUZZER: now also BZ1.1 (+)
- new net SERIAL_CONNECTOR: D1.3 (G), SerialConnect1.4 (Pin_4)
Other:
- moved on the sheet: LoRa_Radio1, SensorBoard1
