File: PCBs/Frame PCB v3/Frame PCB v3.kicad_pcb (KiCad board)
At the start: 2 copper layers, 78 x 40.6 mm, 16 parts, among them J1 Nichrome 1, J2 Nichrome 2, J3 Battery in, J6 Switch, q1 Voltage regulator

Commit message: updated PCBS
Parts:
- removed SensorBoard1, VehiclePowerOn1: I2C Connector, Connector_JST:JST_XH_B4B-XH-A_1x04_P2.50mm_Vertical
- added J10: Nichrome, Connector_JST:JST_XH_B2B-XH-A_1x02_P2.50mm_Vertical, F.Cu at (121.3, 73.8)
- added J11: Nichrome, Connector_JST:JST_XH_B2B-XH-A_1x02_P2.50mm_Vertical, F.Cu at (121.2, 82.2)
- added J5: BayConnector, Connector_JST:JST_XH_B4B-XH-A_1x04_P2.50mm_Vertical, F.Cu at (171.5, 80.2)
- added Q5: Nichrome, Package_TO_SOT_THT:TO-220-3_Vertical, F.Cu at (134.8, 83.0)
- added Q6: Nichrome, Package_TO_SOT_THT:TO-220-3_Vertical, F.Cu at (142.5, 83.1)
- moved J1 13.2 mm to (149.2, 78.0), turned to -90 degrees
- moved J2 8.52 mm to (156.8, 78.4), turned to -90 degrees
- moved R2 6.98 mm to (168.7, 86.2)
- moved R1 5.72 mm to (162.6, 86.3)
- moved BZ1 4.94 mm to (178.9, 81.2)
- moved Teensy4.1 2.36 mm to (158.1, 65.5)
- moved H3 1.77 mm to (190.0, 91.5)
- moved H1 1.45 mm to (190.4, 58.5)
- moved H2 1.24 mm to (121.5, 59.0)
Connections:
- Teensy4.1 pad 32: VehicleSwitch -> unconnected-(Teensy4.1-A17-Pad32)
- Teensy4.1 pad 5: unconnected-(Teensy4.1-PWM-Pad5) -> VehicleOn
Routing:
- net VehicleSwitch: track 49.1 -> 0.00 mm
- net SDA: track 59.7 -> 96.5 mm, vias 0 -> 1
- net VehicleRX: track 48.5 -> 17.9 mm
- net SCL: track 62.4 -> 93.0 mm, vias 1 -> 2
- net VehicleOn: track 0.00 -> 25.3 mm
- net VehicleTX: track 45.7 -> 23.0 mm
- net Net-(J11-Pin_2): track 0.00 -> 21.3 mm, vias 0 -> 1
- net Nichrome1: track 8.95 -> 26.2 mm
- net Nichrome2: track 11.4 -> 27.8 mm, vias 0 -> 1
- net Net-(J10-Pin_2): track 0.00 -> 13.7 mm
- net +5V: track 61.5 -> 68.0 mm
- net BuzzerPin: track 33.5 -> 38.9 mm, vias 0 -> 1
- net Net-(J3-Pin_1): track 13.2 -> 10.4 mm
- net +9V: track 33.8 -> 31.2 mm
Other:
- board size 78 x 40.6 mm -> 76 x 39.3 mm
- board text added: "TRT Payload Frame Board v3.1"
- board text removed: "TRT Payload Frame Board v3.0"
- board text removed: "V RX"
- board text removed: "V TX"

Commit message: updated pcb hole spacing
Parts:
- moved H2 71.0 mm to (192.5, 58.0)
- moved H1 71.0 mm to (119.5, 58.0)
- moved H3 2.66 mm to (192.5, 92.4)
- moved H4 1.82 mm to (119.5, 92.6)
Other:
- board size 76 x 39.3 mm -> 78 x 40 mm

Commit message: fixed traces
Routing:
- net Net-(J11-Pin_2): track 21.3 -> 24.6 mm
Other:
- board text removed: "3.3V+"
- board text removed: "SCL"
- board text removed: "SDA"
Changed lines of the file:
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@@
-	)
-	(gr_text "GND"
-		(at 162.56 75.184 0)
-		(layer "F.SilkS")
-		(effects
-			(font
-				(size 0.5 0.5)
-				(thickness 0.1)
-			)
-			(justify left bottom)
-		)
 	)
 	(gr_text "GND"
@@
 		)
 	)
-	(gr_text "SCL"
-		(at 159.766 75.184 0)
-		(layer "F.SilkS")
-		(effects
-			(font
-				(size 0.5 0.5)
-				(thickness 0.1)
-			)
-			(justify left bottom)
-		)
-	)
 	(gr_text "PWR"
 		(at 144.78 75.438 0)
@@
 	(gr_text "GND"
 		(at 186.1 79.7 0)
-		(layer "F.SilkS")
-		(effects
-			(font
-				(size 0.5 0.5)
-				(thickness 0.1)
-			)
-			(justify left bottom)
-		)
-	)
-	(gr_text "3.3V+"
-		(at 154.432 75.184 0)
-		(layer "F.SilkS")
-		(effects
-			(font
-				(size 0.5 0.5)
-				(thickness 0.1)
-			)
-			(justify left bottom)
-		)
-	)
-	(gr_text "SDA"
-		(at 157.226 75.184 0)
 		(layer "F.SilkS")
 		(effects
@@
 	)
 	(segment
-		(start 134.75 81.7758)
-		(end 135.3141 81.7758)
+		(start 134.75 83.03)
+		(end 134.75 82.5678)
 		(width 0.2)
 		(layer "B.Cu")
@@
 	)
 	(segment
-		(start 134.75 83.03)
-		(end 134.75 81.7758)
+		(start 134.75 82.5678)
+		(end 135.3725 81.9453)
 		(width 0.2)
 		(layer "B.Cu")
@@
 	)
 	(segment
+		(start 137.891108 89.481)
+		(end 138 89.481)
+		(width 0.5)
+		(layer "F.Cu")
+		(net 12)
+	)
+	(segment
+		(start 134.75 77.95)
+		(end 131.628 77.95)
+		(width 0.5)
+		(layer "F.Cu")
+		(net 12)
+	)
+	(segment
+		(start 134.8 78)
+		(end 134.75 77.95)
+		(width 0.5)
+		(layer "F.Cu")
+		(net 12)
+	)
+	(segment
+		(start 137.891108 92.383)
+		(end 137.129 91.620892)
+		(width 0.5)
+		(layer "F.Cu")
+		(net 12)
+	)
+	(segment
+		(start 138 82.25)
+		(end 142.25 78)
+		(width 0.5)
+		(layer "F.Cu")
+		(net 12)
+	)
+	(segment
+		(start 138 89.481)
+		(end 138 82.25)
+		(width 0.5)
+		(layer "F.Cu")
+		(net 12)
+	)
+	(segment
+		(start 127 73.322)
+		(end 127 59.79)
+		(width 0.5)
+		(layer "F.Cu")
+		(net 12)
+	)
+	(segment
+		(start 138 92.383)
+		(end 137.891108 92.383)
+		(width 0.5)
+		(layer "F.Cu")
+		(net 12)
+	)
+	(segment
+		(start 142.25 78)
+		(end 142.5 78)
+		(width 0.5)
+		(layer "F.Cu")
+		(net 12)
+	)
+	(segment
+		(start 142.5 78)
+		(end 134.8 78)
+		(width 0.5)
+		(layer "F.Cu")
+		(net 12)
+	)
+	(segment
+		(start 138.592 93.084)
+		(end 138 92.492)
+		(width 0.5)
+		(layer "F.Cu")
+		(net 12)
+	)
+	(segment
+		(start 154.178 90.861)
+		(end 151.955 93.084)
+		(width 0.5)
+		(layer "F.Cu")
+		(net 12)
+	)
+	(segment
+		(start 138 92.492)
+		(end 138 92.383)
+		(width 0.5)
+		(layer "F.Cu")
+		(net 12)
+	)
+	(segment
+		(start 127 59.79)
+		(end 128.88 57.91)
+		(width 0.5)
+		(layer "F.Cu")
+		(net 12)
+	)
+	(segment
+		(start 137.129 91.620892)
+		(end 137.129 90.243108)
+		(width 0.5)
+		(layer "F.Cu")
+		(net 12)
+	)
+	(segment
 		(start 151.955 93.084)
 		(end 138.592 93.084)
@@
 	)
 	(segment
-		(start 134.75 77.95)
-		(end 131.628 77.95)
-		(width 0.5)
-		(layer "F.Cu")
-		(net 12)
-	)
-	(segment
-		(start 137.129 83.371)
-		(end 142.5 78)
-		(width 0.5)
-		(layer "F.Cu")
-		(net 12)
-	)
-	(segment
-		(start 134.8 78)
-		(end 134.75 77.95)
-		(width 0.5)
-		(layer "F.Cu")
-		(net 12)
-	)
-	(segment
-		(start 127 73.322)
-		(end 127 59.79)
-		(width 0.5)
-		(layer "F.Cu")
-		(net 12)
-	)
-	(segment
-		(start 137.129 91.6209)
-		(end 137.129 83.371)
-		(width 0.5)
-		(layer "F.Cu")
-		(net 12)
-	)
-	(segment
-		(start 142.5 78)
-		(end 134.8 78)
-		(width 0.5)
-		(layer "F.Cu")
-		(net 12)
-	)
-	(segment
-		(start 127 59.79)
-		(end 128.88 57.91)
-		(width 0.5)
-		(layer "F.Cu")
-		(net 12)
-	)
-	(segment
-		(start 138.592 93.084)
-		(end 137.129 91.6209)
-		(width 0.5)
-		(layer "F.Cu")
-		(net 12)
-	)
-	(segment
-		(start 154.178 90.861)
-		(end 151.955 93.084)
+		(start 137.129 90.243108)
+		(end 137.891108 89.481)
 		(width 0.5)
 		(layer "F.Cu")
@@
 		(start 131.6167 80.49)
 		(end 134.75 80.49)
-		(width 0.2)
+		(width 0.5)
 		(layer "B.Cu")
 		(net 28)
@@
 		(start 123.8 73.825)
 		(end 124.9517 73.825)
-		(width 0.2)
+		(width 0.5)
 		(layer "B.Cu")
 		(net 28)
@@
 		(start 124.9517 73.825)
 		(end 131.6167 80.49)
-		(width 0.2)
+		(width 0.5)
 		(layer "B.Cu")
 		(net 28)
@@
 	)
 	(segment
-		(start 136.6848 81.7758)
+		(start 137.299 83.3355)
+		(end 137.299 81.1616)
+		(width 0.5)
+		(layer "F.Cu")
+		(net 53)
+	)
+	(segment
+		(start 137.299 81.1616)
 		(end 139.0313 79.4293)
-		(width 0.2)
-		(layer "F.Cu")
-		(net 53)
-	)
-	(segment
-		(start 124.8517 82.25)
-		(end 125.3259 81.7758)
-		(width 0.2)
-		(layer "F.Cu")
-		(net 53)
-	)
-	(segment
-		(start 125.3259 81.7758)
-		(end 136.6848 81.7758)
-		(width 0.2)
+		(width 0.5)
 		(layer "F.Cu")
 		(net 53)
@@
 		(start 123.7 82.25)
 		(end 124.8517 82.25)
-		(width 0.2)
+		(width 0.5)
+		(layer "F.Cu")
+		(net 53)
+	)
+	(segment
+		(start 124.8517 82.25)
+		(end 128.1017 85.5)
+		(width 0.5)
+		(layer "F.Cu")
+		(net 53)
+	)
+	(segment
+		(start 135.1345 85.5)
+		(end 137.299 83.3355)
+		(width 0.5)
+		(layer "F.Cu")
+		(net 53)
+	)
+	(segment
+		(start 128.1017 85.5)
+		(end 135.1345 85.5)
+		(width 0.5)
 		(layer "F.Cu")
 		(net 53)
@@
 	)
 	(segment
-		(start 142.5 80.54)
-		(end 142.5 79.2858)
-		(width 0.2)
-		(layer "B.Cu")
-		(net 53)
-	)
-	(segment
-		(start 139.1748 79.2858)
-		(end 142.5 79.2858)
-		(width 0.2)
-		(layer "B.Cu")
-		(net 53)
-	)
-	(segment
 		(start 139.0313 79.4293)
 		(end 139.1748 79.2858)
@@
 		(layer "B.Cu")
 		(net 53)
+	)
+	(segment
+		(start 140.142 80.54)
+		(end 139.0313 79.4293)
+		(width 0.5)
+		(layer "B.Cu")
+		(net 53)
+	)
+	(segment
+		(start 142.5 80.54)
+		(end 140.142 80.54)
+		(width 0.5)
+		(layer "B.Cu")
+		(net 53)
