File: PCBs/TADPOL PCB v2/TADPOL PCB v2.kicad_sch (KiCad schematic)
At the start: 23 parts, among them J1 Lora Radio, J10 Nichrome, J11 Battery In, J13 Bypass, J2 Magnetic Connector, J3 Live Video, J4 I2C Connector, J5 Telemetry GPIO, J6 Telemetry Data, J7 Servo 1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

Commit message: fixed traces
Connections:
- net Nichrome_1: now also Teensy4.1.43 (PWM)
Changed lines of the file:
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@@
+		)
+	)
+	(global_label "Nichrome_1"
+		(shape input)
+		(at 153.67 34.29 0)
+		(fields_autoplaced yes)
+		(effects
+			(font
+				(size 1.27 1.27)
+			)
+			(justify left)
+		)
+		(property "Intersheetrefs" "${INTERSHEET_REFS}"
+			(at 167.7223 34.29 0)
+			(effects
+				(font
+					(size 1.27 1.27)
+				)
+				(justify left)
+				(hide yes)
+			)
 		)
 	)

Commit message: fixed Gaia Board
Parts:
- removed J10: Nichrome, Connector_JST:JST_XH_B2B-XH-A_1x02_P2.50mm_Vertical, symbol Connector:Conn_01x02_Socket
- removed J9: Servo 3, Connector_JST:JST_XH_B3B-XH-A_1x03_P2.50mm_Vertical, symbol Connector:Conn_01x03_Socket
- removed Q3: Vehicle On, Package_TO_SOT_THT:TO-220-3_Vertical, symbol Transistor_FET:IRLZ44N
- removed Q4: Vehicle Off, Package_TO_SOT_THT:TO-220-3_Vertical, symbol Transistor_FET:IRLZ44N
- removed Q5: Nichrome, Package_TO_SOT_THT:TO-220-3_Vertical, symbol Transistor_FET:IRLZ44N
- added J12: Vehicle Off, Connector_JST:JST_XH_B2B-XH-A_1x02_P2.50mm_Vertical, symbol Connector:Conn_01x02_Socket
- J4: value I2C Connector -> Sensor Board
Connections:
- net +5V: now also J13.1 (Pin_1), K2.21, K2.B1; no longer VoltRegulator5V1.3 (OUT)
- net GND: now also K2.A2, J12.2 (Pin_2); no longer K2.A1, K2.B2
- net VIN: now also VoltRegulator5V1.1 (IN); no longer J13.2 (Pin_2), K2.24
- net Vehicle_Off: now also K2.B2, J12.1 (Pin_1); no longer Teensy4.1.44 (PWM)
- net Vehicle_On: now also K2.A1
- new net: J13.2 (Pin_2), K2.24, VoltRegulator5V1.3 (OUT)
Other:
- moved on the sheet: J13, VoltRegulator5V1
