File: PCBs/GAIA PCB v2.0/GAIA PCB v2.0.kicad_sch (KiCad schematic)
At the start: 17 parts, among them J1 Servo1, J10 Sensor_Board, J11 Vehicle_On, J12 Vehicle_Off, J13 Battery, J14 Bypass_Switch, J2 Servo2, J3 Servo3, J4 Servo4, J5 Servo5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

Commit message: pcb updates
Parts:
- added H1, H2, H3, H4: MountingHole, MountingHole:MountingHole_3.2mm_M3, symbol Mechanical:MountingHole
- added J15: RC_Control, Connector_JST:JST_XH_B3B-XH-A_1x03_P2.50mm_Vertical, symbol Connector:Conn_01x03_Socket
- J1, J11, J12, J2, J3, J4, J5, J6, J7: footprint (none) -> Connector_JST:JST_XH_B3B-XH-A_1x03_P2.50mm_Vertical
- J10, J8: footprint (none) -> Connector_JST:JST_XH_B4B-XH-A_1x04_P2.50mm_Vertical
- J13, J14: footprint (none) -> Connector_JST:JST_XH_B2B-XH-A_1x02_P2.50mm_Vertical
- J9: footprint (none) -> Connector_JST:JST_XH_B5B-XH-A_1x05_P2.50mm_Vertical
- Volt_Regulator1: renamed from U1; footprint (none) -> Package_TO_SOT_THT:TO-220-3_Vertical
- renumbered K1 to Relay1
Connections:
- net +5V: now also J15.2 (Pin_2)
- net GND: now also J15.3 (Pin_3)
- net PWM_RC: now reaches Teensy4.1.10 (PWM)
- net PWM_RC: now also J15.1 (Pin_1)
