File: PCBs/CNC_PCB/CNC PCB.kicad_sch (KiCad schematic)
At the start: 20 parts, among them J1 Conn_01x02_Pin, J2 Conn_01x02_Pin, J3 Conn_01x02_Pin, J4 Conn_01x02_Pin, U1 BMI088, U2 SN74LVC1T45DBV, U3 MLX90393SLW-ABA-011-RE, U4 L7805CV, U5 MS560702BA03-50

Commit message: Fix Teensy CNC control file loading and launch sequencing
Parts:
- removed BZ1: Buzzer, Buzzer_Beeper:PKMCS0909E4000-R1_MUR, symbol Device:Buzzer
- removed C3, C4: 100nF, Capacitor_SMD:C_0603_1608Metric, symbol Device:C
- removed J2, J3: Conn_01x02_Pin, Connector_JST:JST_XH_B2B-XH-A_1x02_P2.50mm_Vertical, symbol Connector:Conn_01x02_Pin
- removed Teensy4.2: (no value), footprints:Teensy_4.1_Compact, symbol Amplifier_Audio:Teensy4.1
- removed U2: SN74LVC1T45DBV, footprints:SOT-563_DIO, symbol Logic_LevelTranslator:SN74LVC1T45DBV
- removed U3: MLX90393SLW-ABA-011-RE, footprints:QFN-16_MLX90393_MEL, symbol Amplifier_Audio:MLX90393SLW-ABA-011-RE
- removed U4: L7805CV, footprints:L7805CV, symbol Amplifier_Audio:L7805CV
- removed U5: MS560702BA03-50, footprints:SON8_MS5611_TEC, symbol Amplifier_Audio:MS560702BA03-50
- added J5: Conn_01x04, Connector_JST:JST_XH_B4B-XH-AM_1x04_P2.50mm_Vertical, symbol Connector_Generic:Conn_01x04
- added Teensy4.1: (no value), boards:Teensy_4.1, symbol Teensy4.1:Teensy_4.1
- added U2: TXB0104D, D14, symbol TXB0104D:TXB0104D
- added U3: MLX90393SLW-ABA-011-RE, QFN-16_MLX90393_MEL, symbol MLX90393SLW-ABA-111-SP:MLX90393SLW-ABA-011-RE
- added U4, U5: MS561101BA03-50, SON8_MS5611_TEC, symbol MS561101BA03-50:MS561101BA03-50
- R2, R3: value 10KΩ -> 4.7KΩ
Connections:
- net 3.3V: now also Teensy4.1.45 (3.3V), U2.1 (VCCA), U2.8 (OE), U3.15 (VDD), U3.2 (SENB/CS), U3.8 (VDD_IO), U5.1 (VDD), U5.2 (PS)
- net 5V: now also J5.3 (Pin_3), Teensy4.1.47 (Vin), U2.14 (VCCB)
- net ArduinoTx: now also J5.1 (Pin_1), U2.12 (B2)
- net BuzzerPWM: now also Teensy4.1.20 (TX7)
- net ESCData: now also Teensy4.1.44 (PWM)
- net GND: now also J5.4 (Pin_4), Teensy4.1.0 (GND), U2.10 (B4), U2.11 (B3), U2.4 (A3), U2.5 (A4), U2.6 (NC), U2.7 (GND), U2.9 (NC), U3.11 (A1), U3.12 (A0), U3.13 (VSS), U3.17 (GND), U5.3 (GND), U5.4 (CSB)
- net SCL: now also Teensy4.1.40 (SCL), U3.3 (SCL/SCLK), U5.8 (SCLK)
- net SDA: now also Teensy4.1.39 (SDA), U3.5 (SDA/MOSI), U5.7 (SDI/SDA)
- net TeensyRx: now also Teensy4.1.25 (RX8), U2.3 (A2)
- net TeensyTx: now also Teensy4.1.26 (TX8), U2.2 (A1)
- new net ArduinoRx: J5.2 (Pin_2), U2.13 (B1)
